Commit message: xacro initial changes

File: universal_robot/ur_description/urdf/inc/ur_common.xacro (robot description, xacro)
@@ -62,4 +62,8 @@
     <xacro:property name="wrist_3_velocity_limit" value="${sec_limits['wrist_3']['max_velocity']}" scope="parent"/>
     <xacro:property name="wrist_3_effort_limit" value="${sec_limits['wrist_3']['max_effort']}" scope="parent"/>
+    <xacro:property name="prism_lower_limit" value="${sec_limits['wrist_3']['min_position']}" scope="parent"/>
+    <xacro:property name="prism_upper_limit" value="${sec_limits['prism']['max_position']}" scope="parent"/>
+    <xacro:property name="prism_velocity_limit" value="${sec_limits['prism']['max_velocity']}" scope="parent"/>
+    <xacro:property name="prism_effort_limit" value="${sec_limits['prism']['max_effort']}" scope="parent"/>
     <!-- DH PARAMETERS -->
     <xacro:property name="d1" value="${sec_dh_parameters['d1']}" scope="parent"/>
@@ -106,4 +110,10 @@
     <xacro:property name="wrist_3_pitch" value="${sec_kinematics['wrist_3']['pitch']}" scope="parent"/>
     <xacro:property name="wrist_3_yaw" value="${sec_kinematics['wrist_3']['yaw']}" scope="parent"/>
+    <xacro:property name="prism_x" value="${sec_kinematics['prism']['x']}" scope="parent"/>
+    <xacro:property name="prism_y" value="${sec_kinematics['prism']['y']}" scope="parent"/>
+    <xacro:property name="prism_z" value="${sec_kinematics['prism']['z']}" scope="parent"/>
+    <xacro:property name="prism_roll" value="${sec_kinematics['prism']['roll']}" scope="parent"/>
+    <xacro:property name="prism_pitch" value="${sec_kinematics['prism']['pitch']}" scope="parent"/>
+    <xacro:property name="prism_yaw" value="${sec_kinematics['prism']['yaw']}" scope="parent"/>
     <!-- OFFSETS -->
     <xacro:property name="shoulder_offset" value="${sec_offsets['shoulder_offset']}" scope="parent"/>
@@ -119,4 +129,5 @@
     <xacro:property name="wrist_2_mass" value="${sec_inertia_parameters['wrist_2_mass']}" scope="parent"/>
     <xacro:property name="wrist_3_mass" value="${sec_inertia_parameters['wrist_3_mass']}" scope="parent"/>
+    <xacro:property name="prism_mass" value="${sec_inertia_parameters['prism_mass']}" scope="parent"/>
     <!-- link inertia parameter -->
     <xacro:property name="intertia_links" value="${sec_inertia_parameters['links']}" scope="parent"/>
@@ -135,4 +146,6 @@
     <xacro:property name="wrist_3_inertia_radius" value="${intertia_links['wrist_3']['radius']}" scope="parent"/>
     <xacro:property name="wrist_3_inertia_length" value="${intertia_links['wrist_3']['length']}" scope="parent"/>
+    <xacro:property name="prism_inertia_radius" value="${intertia_links['prism']['radius']}" scope="parent"/>
+    <xacro:property name="prism_inertia_length" value="${intertia_links['prism']['length']}" scope="parent"/>
     <!-- center of mass -->
     <xacro:property name="prop_shoulder_cog" value="${sec_inertia_parameters['center_of_mass']['shoulder_cog']}" scope="parent"/>
@@ -142,4 +155,5 @@
     <xacro:property name="prop_wrist_2_cog" value="${sec_inertia_parameters['center_of_mass']['wrist_2_cog']}" scope="parent"/>
     <xacro:property name="prop_wrist_3_cog" value="${sec_inertia_parameters['center_of_mass']['wrist_3_cog']}" scope="parent"/>
+    <xacro:property name="prop_prism_cog" value="${sec_inertia_parameters['center_of_mass']['prism_cog']}" scope="parent"/>
     <xacro:property name="shoulder_cog" value="${prop_shoulder_cog['x']} ${prop_shoulder_cog['y']} ${prop_shoulder_cog['z']}" scope="parent"/>
     <xacro:property name="upper_arm_cog" value="${prop_upper_arm_cog['x']} ${prop_upper_arm_cog['y']} ${prop_upper_arm_cog['z']}" scope="parent"/>
@@ -148,4 +162,5 @@
     <xacro:property name="wrist_2_cog" value="${prop_wrist_2_cog['x']} ${prop_wrist_2_cog['y']} ${prop_wrist_2_cog['z']}" scope="parent"/>
     <xacro:property name="wrist_3_cog" value="${prop_wrist_3_cog['x']} ${prop_wrist_3_cog['y']} ${prop_wrist_3_cog['z']}" scope="parent"/>
+    <xacro:property name="prism_cog" value="${prop_prism_cog['x']} ${prop_prism_cog['y']} ${prop_prism_cog['z']}" scope="parent"/>
     <!-- cylinder radius -->
     <xacro:property name="shoulder_radius" value="${sec_inertia_parameters['shoulder_radius']}" scope="parent"/>
@@ -154,4 +169,5 @@
     <xacro:property name="forearm_radius" value="${sec_inertia_parameters['forearm_radius']}" scope="parent"/>
     <xacro:property name="wrist_radius" value="${sec_inertia_parameters['wrist_radius']}" scope="parent"/>
+    <xacro:property name="prism_radius" value="${sec_inertia_parameters['prism_radius']}" scope="parent"/>
     <!-- Mesh files -->
     <xacro:property name="base_mesh" value="${sec_mesh_files['base']}"/>
@@ -193,4 +209,10 @@
     <xacro:property name="wrist_3_collision_mesh" value="${wrist_3_mesh['collision']['mesh']}" scope="parent"/>
     <xacro:property name="wrist_3_visual_offset" value="${wrist_3_mesh['visual_offset']}" scope="parent"/>
+    <xacro:property name="prism_mesh" value="${sec_mesh_files['prism']}"/>
+    <xacro:property name="prism_visual_mesh" value="${prism_mesh['visual']['mesh']}" scope="parent"/>
+    <xacro:property name="prism_visual_material_name" value="${prism_mesh['visual']['material']['name']}" scope="parent"/>
+    <xacro:property name="prism_visual_material_color" value="${prism_mesh['visual']['material']['color']}" scope="parent"/>
+    <xacro:property name="prism_collision_mesh" value="${prism_mesh['collision']['mesh']}" scope="parent"/>
+    <xacro:property name="prism_visual_offset" value="${prism_mesh['visual_offset']}" scope="parent"/>
   </xacro:macro>
 </robot>
