Commit message: pruebas construct

File: universal_robot/kuka_kr20_description/urdf/kr20.xacro (robot description, xacro)
@@ -48,26 +48,15 @@
     <material>Gazebo/Orange</material>
   </gazebo>
-  <gazebo reference="${gripper_name}">
-    <material>Gazebo/Black</material>
+  <gazebo reference="${link_06_name}">
+    <material>Gazebo/Orange</material>
   </gazebo>
-  <gazebo reference="gripper_left">
-    <material>Gazebo/White</material>
-    <mu1>1.0</mu1>
-    <mu2>1.0</mu2>
-    <kp>1000000.0</kp>
-    <kd>1.0</kd>
-    <minDepth>0.001</minDepth>
-    <!--maxVel>0.1</maxVel>
-    <fdir1>1 0 0</fdir1-->
+  <gazebo reference="${link_07_name}">
+    <material>Gazebo/Orange</material>
   </gazebo>
-  <gazebo reference="gripper_right">
-    <material>Gazebo/White</material>
-    <mu1>1.0</mu1>
-    <mu2>1.0</mu2>
-    <kp>1000000.0</kp>
-    <kd>1.0</kd>
-    <minDepth>0.001</minDepth>
-    <!--maxVel>0.1</maxVel>
-    <fdir1>1 0 0</fdir1-->
+  <gazebo reference="${link_08_name}">
+    <material>Gazebo/Orange</material>
+  </gazebo>
+  <gazebo reference="${link_09_name}">
+    <material>Gazebo/Orange</material>
   </gazebo>
   <!-- BEGIN - Robot description -->

File: universal_robot/kuka_kr20_description/urdf/robot_parameters.xacro (robot description, xacro)
@@ -7,5 +7,7 @@
   <xacro:property name="link_04_name" value="link04" />
   <xacro:property name="link_05_name" value="link05" />
-  <xacro:property name="gripper_name" value="gripper" />
+  <xacro:property name="link_06_name" value="link06" />
+  <xacro:property name="link_07_name" value="link07" />
+  <xacro:property name="link_08_name" value="linkef" />
   <xacro:property name="camera_z" value="1.7" />
   <xacro:property name="camera_y" value="1.0" />

Commit message: xacro completed

File: universal_robot/kuka_kr20_description/urdf/kr20.xacro (robot description, xacro)
@@ -19,5 +19,5 @@
               iyy="13.235" iyz="0"
               izz="9.655"
-              meshfile="package://kuka_kr20_description/meshes/base.stl"
+              meshfile="package://kuka_kr20_description/meshes/base_link.stl"
               meshscale="0.001 0.001 0.001" />
   <material name="Orange">
@@ -57,121 +57,108 @@
     <material>Gazebo/Orange</material>
   </gazebo>
-  <gazebo reference="${link_09_name}">
-    <material>Gazebo/Orange</material>
-  </gazebo>
   <!-- BEGIN - Robot description -->
-  <xacro:m_joint name="${link_00_name}__${link_01_name}" type="revolute"
+  <xacro:m_joint name="q1" type="revolute"
            axis_xyz="0 0 1"
-           origin_rpy="0 0 0" origin_xyz="0 0 0.3"
+           origin_rpy="0 0 0" origin_xyz="0 0 1.08725"
            parent="${link_00_name}" child="${link_01_name}"
-           limit_e="1000" limit_l="-3" limit_u="3" limit_v="0.5" />
+           limit_e="1000" limit_l="-3.14" limit_u="3.14" limit_v="0.5" />
   <xacro:m_link_mesh name="${link_01_name}" color="Orange"
-              origin_rpy="1.5708 0 -1.5708" origin_xyz="0 0 0"
+              origin_rpy="1.5708 0 0" origin_xyz="0 0 -0.12725"
               mass="157.633"
               ixx="13.235" ixy="0" ixz="0"
               iyy="13.235" iyz="0"
               izz="9.655"
-              meshfile="package://kuka_kr20_description/meshes/link1.stl"
+              meshfile="package://kuka_kr20_description/meshes/Link1.stl"
               meshscale="0.001 0.001 0.001" />
-  <xacro:m_joint name="${link_01_name}__${link_02_name}" type="revolute"
-           axis_xyz="0 1 0"
-           origin_rpy="0 0 0" origin_xyz="0.160 -0.095 0.220"
+  <xacro:m_joint name="q2" type="prismatic"
+           axis_xyz="0 0 1"
+           origin_rpy="0 1.5708 0" origin_xyz="0 -0.115 0"
            parent="${link_01_name}" child="${link_02_name}"
-           limit_e="1000" limit_l="-1.5708" limit_u="1.7453" limit_v="0.5" />
-  <xacro:m_link_mesh name="${link_02_name}" color="Orange"
-              origin_rpy="1.5708 0 1.5708" origin_xyz="0 0 0"
-              mass="10"
-              ixx="10" ixy="0" ixz="0"
-              iyy="10" iyz="0"
-              izz="10"
-              meshfile="package://kuka_kr20_description/meshes/link2.stl"
+           limit_e="1000" limit_l="0.13" limit_u="0.5" limit_v="0.5" />
+  <xacro:m_link_mesh name="${link_02_name}" color="Grey"
+              origin_rpy="0 0 -1.5708" origin_xyz="0 0.11 0"
+              mass="157.633"
+              ixx="13.235" ixy="0" ixz="0"
+              iyy="13.235" iyz="0"
+              izz="9.655"
+              meshfile="package://kuka_kr20_description/meshes/Link2.stl"
               meshscale="0.001 0.001 0.001" />
-  <xacro:m_joint name="${link_02_name}__${link_03_name}" type="revolute"
-           axis_xyz="0 -1 0"
-           origin_rpy="0 0 0" origin_xyz="0.00 -0.01 0.780"
+  <xacro:m_joint name="q3" type="revolute"
+           axis_xyz="0 0 1"
+           origin_rpy="0 0 0" origin_xyz="0 0 0.2835"
            parent="${link_02_name}" child="${link_03_name}"
-           limit_e="1000" limit_l="-2" limit_u="2" limit_v="0.5" />
+           limit_e="1000" limit_l="-2.15" limit_u="2.15" limit_v="0.5" />
   <xacro:m_link_mesh name="${link_03_name}" color="Orange"
-              origin_rpy="1.5708 0 -1.5708" origin_xyz="0 0 0"
-              mass="7"
-              ixx="5" ixy="0" ixz="0"
-              iyy="5" iyz="0"
-              izz="5"
-              meshfile="package://kuka_kr20_description/meshes/link3.stl"
+              origin_rpy="0 0 -1.5708" origin_xyz="0 0 -0.08675"
+              mass="157.633"
+              ixx="13.235" ixy="0" ixz="0"
+              iyy="13.235" iyz="0"
+              izz="9.655"
+              meshfile="package://kuka_kr20_description/meshes/Link3.stl"
               meshscale="0.001 0.001 0.001" />
-  <xacro:m_joint name="${link_03_name}__${link_04_name}" type="revolute"
-           axis_xyz="1 0 0"
-           origin_rpy="0 0 0" origin_xyz="0.700 0.105 0.150"
+  <xacro:m_joint name="q4" type="revolute"
+           axis_xyz="0 0 1"
+           origin_rpy="0 0 0" origin_xyz="0 -0.656 -0.13225"
            parent="${link_03_name}" child="${link_04_name}"
-           limit_e="1000" limit_l="-3.0" limit_u="3.0" limit_v="0.5" />
-  <xacro:m_link_mesh name="${link_04_name}" color="Orange"
-              origin_rpy="1.5708 0 1.5708" origin_xyz="0 0 0"
-              mass="2"
-              ixx="1" ixy="0" ixz="0"
-              iyy="1" iyz="0"
-              izz="1"
-              meshfile="package://kuka_kr20_description/meshes/link4.stl"
+           limit_e="1000" limit_l="-3.14" limit_u="3.14" limit_v="0.5" />
+  <xacro:m_link_mesh name="${link_04_name}" color="Grey"
+              origin_rpy="0 0 -1.5708" origin_xyz="0 0 -0.06425"
+              mass="157.633"
+              ixx="13.235" ixy="0" ixz="0"
+              iyy="13.235" iyz="0"
+              izz="9.655"
+              meshfile="package://kuka_kr20_description/meshes/Link4.stl"
               meshscale="0.001 0.001 0.001" />
-  <xacro:m_joint name="${link_04_name}__${link_05_name}" type="revolute"
-           axis_xyz="0 -1 0"
-           origin_rpy="0 0 0" origin_xyz="0.155 0.000 0.000"
+  <xacro:m_joint name="q5" type="revolute"
+           axis_xyz="0 0 1"
+           origin_rpy="0 0 0" origin_xyz="0 -0.531 0.1565"
            parent="${link_04_name}" child="${link_05_name}"
-           limit_e="1000" limit_l="-3.0" limit_u="3.0" limit_v="0.5" />
+           limit_e="1000" limit_l="-3.14" limit_u="3.14" limit_v="0.5" />
   <xacro:m_link_mesh name="${link_05_name}" color="Orange"
-              origin_rpy="1.5708 0 1.5708" origin_xyz="0 0 0"
-              mass="2"
-              ixx="1" ixy="0" ixz="0"
-              iyy="1" iyz="0"
-              izz="1"
-              meshfile="package://kuka_kr20_description/meshes/link5.stl"
+              origin_rpy="0 -1.5708 1.5708" origin_xyz="0 0 0"
+              mass="157.633"
+              ixx="13.235" ixy="0" ixz="0"
+              iyy="13.235" iyz="0"
+              izz="9.655"
+              meshfile="package://kuka_kr20_description/meshes/Link5.stl"
               meshscale="0.001 0.001 0.001" />
-  <!-- GRIPPER START HERE -->
-  <xacro:m_joint name="${link_05_name}__${gripper_name}" type="revolute"
-           axis_xyz="1 0 0"
-           origin_rpy="0 0 0" origin_xyz="0.115 0 0"
-           parent="${link_05_name}" child="${gripper_name}"
-           limit_e="1000" limit_l="-1.57" limit_u="1.57" limit_v="0.5" />
-  <xacro:m_link_mesh name="${gripper_name}" color="Black"
-              origin_rpy="1.5708 0 1.5708" origin_xyz="0 0 0"
-              mass="1"
-              ixx="1" ixy="0" ixz="0"
-              iyy="1" iyz="0"
-              izz="1"
-              meshfile="package://kuka_kr20_description/meshes/gripper_base.stl"
+   <xacro:m_joint name="q6" type="revolute"
+           axis_xyz="0 0 1"
+           origin_rpy="1.5708 0 0" origin_xyz="0 -0.1605 0"
+           parent="${link_05_name}" child="${link_06_name}"
+           limit_e="1000" limit_l="-3.14" limit_u="3.14" limit_v="0.5" />
+  <xacro:m_link_mesh name="${link_06_name}" color="Grey"
+              origin_rpy="0 -1.5708 1.5708" origin_xyz="0 0 -0.0605"
+              mass="157.633"
+              ixx="13.235" ixy="0" ixz="0"
+              iyy="13.235" iyz="0"
+              izz="9.655"
+              meshfile="package://kuka_kr20_description/meshes/Link6.stl"
               meshscale="0.001 0.001 0.001" />
-  <xacro:m_joint name="${gripper_name}__gripper_left" type="prismatic"
-           axis_xyz="1 0 0"
-           origin_rpy="1.5708 0 1.5708" origin_xyz="0.04 0.00 0.000"
-           parent="${gripper_name}" child="gripper_left"
-           limit_e="1000" limit_l="-0.09" limit_u="0.00" limit_v="0.5" />
-  <xacro:m_link_mesh name="gripper_left" color="Grey"
-              origin_rpy="0 0 0" origin_xyz="0 0 0"
-              mass="0.1"
-              ixx="1" ixy="0" ixz="0"
-              iyy="1" iyz="0"
-              izz="1"
-              meshfile="package://kuka_kr20_description/meshes/gripper_left.stl"
+   <xacro:m_joint name="q7" type="revolute"
+           axis_xyz="0 0 1"
+           origin_rpy="-1.5708 0 0" origin_xyz="0 0 0"
+           parent="${link_06_name}" child="${link_07_name}"
+           limit_e="1000" limit_l="-3.14" limit_u="3.14" limit_v="0.5" />
+  <xacro:m_link_mesh name="${link_07_name}" color="Orange"
+              origin_rpy="0 3.1416 0" origin_xyz="0 0 0.088"
+              mass="157.633"
+              ixx="13.235" ixy="0" ixz="0"
+              iyy="13.235" iyz="0"
+              izz="9.655"
+              meshfile="package://kuka_kr20_description/meshes/Link7.stl"
               meshscale="0.001 0.001 0.001" />
-  <xacro:m_joint name="${gripper_name}__gripper_right" type="prismatic"
-           axis_xyz="1 0 0"
-           origin_rpy="1.5708 0 1.5708" origin_xyz="0.04 0.00 0.000"
-           parent="${gripper_name}" child="gripper_right"
-           limit_e="1000" limit_l="0.00" limit_u="0.09" limit_v="0.5" />
-  <xacro:m_link_mesh name="gripper_right" color="Grey"
-              origin_rpy="0 0 0" origin_xyz="0 0 0"
-              mass="0.1"
-              ixx="1" ixy="0" ixz="0"
-              iyy="1" iyz="0"
-              izz="1"
-              meshfile="package://kuka_kr20_description/meshes/gripper_right.stl"
+   <xacro:m_joint name="q8" type="prismatic"
+           axis_xyz="0 0 1"
+           origin_rpy="0 0 0" origin_xyz="0 0 0"
+           parent="${link_07_name}" child="${link_08_name}"
+           limit_e="1000" limit_l="-0.08" limit_u="0.08" limit_v="0.5" />
+  <xacro:m_link_mesh name="${link_08_name}" color="Black"
+              origin_rpy="0 -1.5708 0" origin_xyz="0 0 -0.15"
+              mass="157.633"
+              ixx="13.235" ixy="0" ixz="0"
+              iyy="13.235" iyz="0"
+              izz="9.655"
+              meshfile="package://kuka_kr20_description/meshes/Link_EF.stl"
               meshscale="0.001 0.001 0.001" />
-  <!-- GRIPPER END HERE -->
-  <!-- END - Robot description -->
-  <gazebo>
-    <plugin name="gazebo_ros_control" filename="libgazebo_ros_control.so">
-      <robotSimType>gazebo_ros_control/DefaultRobotHWSim</robotSimType>
-      <robotNamespace>/kr20</robotNamespace>
-      <legacyModeNS>true</legacyModeNS>
-    </plugin>
-  </gazebo>
 </robot>

Commit message: fixed links

File: universal_robot/kuka_kr20_description/urdf/kr20.xacro (robot description, xacro)
@@ -13,6 +13,6 @@
     <origin rpy="0 0 0" xyz="0 0 0"/>
   </joint>
-  <xacro:m_link_mesh name="${link_00_name}" color="Black"
-              origin_rpy="1.5708 0 3.1416" origin_xyz="0 0 0"
+  <xacro:m_link_mesh name="${link_00_name}" color="White"
+              origin_rpy="0 0 0" origin_xyz="0 0 0"
               mass="157.633"
               ixx="13.235" ixy="0" ixz="0"
@@ -21,48 +21,51 @@
               meshfile="package://kuka_kr20_description/meshes/base_link.stl"
               meshscale="0.001 0.001 0.001" />
-  <material name="Orange">
-    <color rgba="0.95 0.5 0.15 1.0"/>
+  <material name="DarkGreen">
+    <color rgba="0 0.36 0.012 1.0"/>
+  </material>
+  <material name="LightGreen">
+    <color rgba="0.82 0.95 0.82 1.0"/>
+  </material>
+  <material name="White">
+    <color rgba="0.96 0.96 0.96 1.0"/>
   </material>
   <material name="Grey">
-    <color rgba="0.7 0.7 0.7 1.0"/>
-  </material>
-  <material name="Black">
-    <color rgba="0.0 0.0 0.0 1.0"/>
+    <color rgba="0.56 0.56 0.56 1.0"/>
   </material>
   <gazebo reference="${link_00_name}">
-    <material>Gazebo/Black</material>
+    <material>Gazebo/White</material>
   </gazebo>
   <gazebo reference="${link_01_name}">
-    <material>Gazebo/Orange</material>
+    <material>Gazebo/Grey</material>
   </gazebo>
   <gazebo reference="${link_02_name}">
-    <material>Gazebo/Orange</material>
+    <material>Gazebo/DarkGreen</material>
   </gazebo>
   <gazebo reference="${link_03_name}">
-    <material>Gazebo/Orange</material>
+    <material>Gazebo/LightGreen</material>
   </gazebo>
   <gazebo reference="${link_04_name}">
-    <material>Gazebo/Orange</material>
+    <material>Gazebo/LightGreen</material>
   </gazebo>
   <gazebo reference="${link_05_name}">
-    <material>Gazebo/Orange</material>
+    <material>Gazebo/LightGreen</material>
   </gazebo>
   <gazebo reference="${link_06_name}">
-    <material>Gazebo/Orange</material>
+    <material>Gazebo/LightGreen</material>
   </gazebo>
   <gazebo reference="${link_07_name}">
-    <material>Gazebo/Orange</material>
+    <material>Gazebo/LightGreen</material>
   </gazebo>
   <gazebo reference="${link_08_name}">
-    <material>Gazebo/Orange</material>
+    <material>Gazebo/Grey</material>
   </gazebo>
   <!-- BEGIN - Robot description -->
   <xacro:m_joint name="q1" type="revolute"
            axis_xyz="0 0 1"
-           origin_rpy="0 0 0" origin_xyz="0 0 1.08725"
+           origin_rpy="0 0 0" origin_xyz="0 0 1.65"
            parent="${link_00_name}" child="${link_01_name}"
            limit_e="1000" limit_l="-3.14" limit_u="3.14" limit_v="0.5" />
-  <xacro:m_link_mesh name="${link_01_name}" color="Orange"
-              origin_rpy="1.5708 0 0" origin_xyz="0 0 -0.12725"
+  <xacro:m_link_mesh name="${link_01_name}" color="Grey"
+              origin_rpy="0 0 0" origin_xyz="0 0 0"
               mass="157.633"
               ixx="13.235" ixy="0" ixz="0"
@@ -72,10 +75,10 @@
               meshscale="0.001 0.001 0.001" />
   <xacro:m_joint name="q2" type="prismatic"
-           axis_xyz="0 0 1"
-           origin_rpy="0 1.5708 0" origin_xyz="0 -0.115 0"
+           axis_xyz="0 1 0"
+           origin_rpy="0 0 0" origin_xyz="0 0.37775 0.089"
            parent="${link_01_name}" child="${link_02_name}"
-           limit_e="1000" limit_l="0.13" limit_u="0.5" limit_v="0.5" />
-  <xacro:m_link_mesh name="${link_02_name}" color="Grey"
-              origin_rpy="0 0 -1.5708" origin_xyz="0 0.11 0"
+           limit_e="1000" limit_l="-0.192" limit_u="0.216" limit_v="0.5" />
+  <xacro:m_link_mesh name="${link_02_name}" color="DarkGreen"
+              origin_rpy="0 0 0" origin_xyz="0 0 0"
               mass="157.633"
               ixx="13.235" ixy="0" ixz="0"
@@ -85,10 +88,10 @@
               meshscale="0.001 0.001 0.001" />
   <xacro:m_joint name="q3" type="revolute"
-           axis_xyz="0 0 1"
-           origin_rpy="0 0 0" origin_xyz="0 0 0.2835"
+           axis_xyz="0 1 0"
+           origin_rpy="0 0 0" origin_xyz="0.115 0.11 0"
            parent="${link_02_name}" child="${link_03_name}"
            limit_e="1000" limit_l="-2.15" limit_u="2.15" limit_v="0.5" />
-  <xacro:m_link_mesh name="${link_03_name}" color="Orange"
-              origin_rpy="0 0 -1.5708" origin_xyz="0 0 -0.08675"
+  <xacro:m_link_mesh name="${link_03_name}" color="LightGreen"
+              origin_rpy="0 0 0" origin_xyz="0 0 0"
               mass="157.633"
               ixx="13.235" ixy="0" ixz="0"
@@ -98,10 +101,10 @@
               meshscale="0.001 0.001 0.001" />
   <xacro:m_joint name="q4" type="revolute"
-           axis_xyz="0 0 1"
-           origin_rpy="0 0 0" origin_xyz="0 -0.656 -0.13225"
+           axis_xyz="0 1 0"
+           origin_rpy="0 0 0" origin_xyz="0.65625 0.0225 0"
            parent="${link_03_name}" child="${link_04_name}"
            limit_e="1000" limit_l="-3.14" limit_u="3.14" limit_v="0.5" />
-  <xacro:m_link_mesh name="${link_04_name}" color="Grey"
-              origin_rpy="0 0 -1.5708" origin_xyz="0 0 -0.06425"
+  <xacro:m_link_mesh name="${link_04_name}" color="LightGreen"
+              origin_rpy="0 0 0" origin_xyz="0 0 0"
               mass="157.633"
               ixx="13.235" ixy="0" ixz="0"
@@ -111,10 +114,10 @@
               meshscale="0.001 0.001 0.001" />
   <xacro:m_joint name="q5" type="revolute"
-           axis_xyz="0 0 1"
-           origin_rpy="0 0 0" origin_xyz="0 -0.531 0.1565"
+           axis_xyz="0 1 0"
+           origin_rpy="0 0 0" origin_xyz=" 0.531 -0.011475 0"
            parent="${link_04_name}" child="${link_05_name}"
            limit_e="1000" limit_l="-3.14" limit_u="3.14" limit_v="0.5" />
-  <xacro:m_link_mesh name="${link_05_name}" color="Orange"
-              origin_rpy="0 -1.5708 1.5708" origin_xyz="0 0 0"
+  <xacro:m_link_mesh name="${link_05_name}" color="LightGreen"
+              origin_rpy="0 0 0" origin_xyz="0 0 0"
               mass="157.633"
               ixx="13.235" ixy="0" ixz="0"
@@ -124,10 +127,10 @@
               meshscale="0.001 0.001 0.001" />
    <xacro:m_joint name="q6" type="revolute"
-           axis_xyz="0 0 1"
-           origin_rpy="1.5708 0 0" origin_xyz="0 -0.1605 0"
+           axis_xyz="1 0 0"
+           origin_rpy="0 0 0" origin_xyz="0.0985 0.1 0"
            parent="${link_05_name}" child="${link_06_name}"
            limit_e="1000" limit_l="-3.14" limit_u="3.14" limit_v="0.5" />
-  <xacro:m_link_mesh name="${link_06_name}" color="Grey"
-              origin_rpy="0 -1.5708 1.5708" origin_xyz="0 0 -0.0605"
+  <xacro:m_link_mesh name="${link_06_name}" color="LightGreen"
+              origin_rpy="0 0 0" origin_xyz="0 0 0"
               mass="157.633"
               ixx="13.235" ixy="0" ixz="0"
@@ -137,10 +140,10 @@
               meshscale="0.001 0.001 0.001" />
    <xacro:m_joint name="q7" type="revolute"
-           axis_xyz="0 0 1"
-           origin_rpy="-1.5708 0 0" origin_xyz="0 0 0"
+           axis_xyz="0 1 0"
+           origin_rpy="0 0 0" origin_xyz="0.0605 0.057 0"
            parent="${link_06_name}" child="${link_07_name}"
            limit_e="1000" limit_l="-3.14" limit_u="3.14" limit_v="0.5" />
-  <xacro:m_link_mesh name="${link_07_name}" color="Orange"
-              origin_rpy="0 3.1416 0" origin_xyz="0 0 0.088"
+  <xacro:m_link_mesh name="${link_07_name}" color="Grey"
+              origin_rpy="0 0 0" origin_xyz="0 0 0"
               mass="157.633"
               ixx="13.235" ixy="0" ixz="0"
@@ -150,10 +153,10 @@
               meshscale="0.001 0.001 0.001" />
    <xacro:m_joint name="q8" type="prismatic"
-           axis_xyz="0 0 1"
-           origin_rpy="0 0 0" origin_xyz="0 0 0"
+           axis_xyz="0 1 0"
+           origin_rpy="0 0 0" origin_xyz="0 -0.092 0"
            parent="${link_07_name}" child="${link_08_name}"
-           limit_e="1000" limit_l="-0.08" limit_u="0.08" limit_v="0.5" />
-  <xacro:m_link_mesh name="${link_08_name}" color="Black"
-              origin_rpy="0 -1.5708 0" origin_xyz="0 0 -0.15"
+           limit_e="1000" limit_l="0" limit_u="0.1" limit_v="0.5" />
+  <xacro:m_link_mesh name="${link_08_name}" color="Grey"
+              origin_rpy="0 0 0" origin_xyz="0 0 0"
               mass="157.633"
               ixx="13.235" ixy="0" ixz="0"
