Commit message: control and corrected DH

File: universal_robot/kuka_kr20_description/urdf/kr20.urdf (robot description, URDF)
Before this commit: robot kr20, 10 links, 9 joints
Links:
- link base: mass 157.633 -> 414.0
- link link01: mass 157.633 -> 24.74
- link link02: mass 157.633 -> 10.88
- link link03: mass 157.633 -> 19.26
- link link04: mass 157.633 -> 9.9
- link link05: mass 157.633 -> 2.38
- link link06: mass 157.633 -> 1.75
- link link07: mass 157.633 -> 0.37
- link linkef: mass 157.633 -> 1.69
Joints:
- joint q1: origin xyz=0 0 1.08725 rpy=1.5708 0 3.1416 -> xyz=0 0 1.65 rpy=0 0 0
- joint q2: axis 0 0 1 -> 0 1 0; limit lower=0.13 upper=0.5 effort=1000 velocity=0.5 -> lower=-0.192 upper=0.216 effort=1000 velocity=0.5; origin xyz=0 -0.115 0 rpy=0 3.1416 0 -> xyz=0 0.37775 0.089 rpy=0 0 0
- joint q3: axis 0 0 1 -> 0 1 0; origin xyz=0 0 0.2835 rpy=0 0 -1.5708 -> xyz=0.115 0.11 0 rpy=0 0 0
- joint q4: axis 0 0 1 -> 0 1 0; origin xyz=0 -0.656 -0.13225 rpy=0 0 -1.5708 -> xyz=0.65625 0.0225 0 rpy=0 0 0
- joint q5: axis 0 0 1 -> 0 1 0; origin xyz=0 -0.531 0.1565 rpy=0 -1.5708 1.5708 -> xyz= 0.531 -0.011475 0 rpy=0 0 0
- joint q6: axis 0 0 1 -> 1 0 0; origin xyz=0 -0.1605 0 rpy=1.5708 -1.5708 0 -> xyz=0.0985 0.1 0 rpy=0 0 0
- joint q7: axis 0 0 1 -> 0 1 0; origin xyz=0 0 0 rpy=-1.5708 0 0 -> xyz=0.0605 0.057 0 rpy=0 0 0
- joint q8: axis 0 0 1 -> 0 1 0; limit lower=-0.08 upper=0.08 effort=1000 velocity=0.5 -> lower=0 upper=0.1 effort=1000 velocity=0.5; origin xyz=0 0 0 rpy=0 -1.5708 0 -> xyz=0 -0.09 0 rpy=0 0 0

File: universal_robot/kuka_kr20_description/urdf/kr20.xacro (robot description, xacro)
@@ -15,8 +15,8 @@
   <xacro:m_link_mesh name="${link_00_name}" color="White"
               origin_rpy="0 0 0" origin_xyz="0 0 0"
-              mass="157.633"
-              ixx="13.235" ixy="0" ixz="0"
-              iyy="13.235" iyz="0"
-              izz="9.655"
+              mass="414.0"
+              ixx="97670000" ixy="0" ixz="0"
+              iyy="97670000" iyz="0"
+              izz="2170000"
               meshfile="package://kuka_kr20_description/meshes/base_link.stl"
               meshscale="0.001 0.001 0.001" />
@@ -68,8 +68,8 @@
   <xacro:m_link_mesh name="${link_01_name}" color="Grey"
               origin_rpy="0 0 0" origin_xyz="0 0 0"
-              mass="157.633"
-              ixx="13.235" ixy="0" ixz="0"
-              iyy="13.235" iyz="0"
-              izz="9.655"
+              mass="24.74"
+              ixx="1430" ixy="84.25" ixz="0.2969"
+              iyy="82.08" iyz="-1.64"
+              izz="1405"
               meshfile="package://kuka_kr20_description/meshes/Link1.stl"
               meshscale="0.001 0.001 0.001" />
@@ -81,8 +81,8 @@
   <xacro:m_link_mesh name="${link_02_name}" color="DarkGreen"
               origin_rpy="0 0 0" origin_xyz="0 0 0"
-              mass="157.633"
-              ixx="13.235" ixy="0" ixz="0"
-              iyy="13.235" iyz="0"
-              izz="9.655"
+              mass="10.88"
+              ixx="67.73" ixy="1.2" ixz="0.184"
+              iyy="59.85" iyz="-0.005"
+              izz="83.55"
               meshfile="package://kuka_kr20_description/meshes/Link2.stl"
               meshscale="0.001 0.001 0.001" />
@@ -94,8 +94,8 @@
   <xacro:m_link_mesh name="${link_03_name}" color="LightGreen"
               origin_rpy="0 0 0" origin_xyz="0 0 0"
-              mass="157.633"
-              ixx="13.235" ixy="0" ixz="0"
-              iyy="13.235" iyz="0"
-              izz="9.655"
+              mass="19.26"
+              ixx="56.06" ixy="-4.0" ixz="0"
+              iyy="1396.0" iyz="0"
+              izz="1404.0"
               meshfile="package://kuka_kr20_description/meshes/Link3.stl"
               meshscale="0.001 0.001 0.001" />
@@ -107,8 +107,8 @@
   <xacro:m_link_mesh name="${link_04_name}" color="LightGreen"
               origin_rpy="0 0 0" origin_xyz="0 0 0"
-              mass="157.633"
-              ixx="13.235" ixy="0" ixz="0"
-              iyy="13.235" iyz="0"
-              izz="9.655"
+              mass="9.9"
+              ixx="17.71" ixy="0.209" ixz="-0.001"
+              iyy="464.8" iyz="0"
+              izz="467.7"
               meshfile="package://kuka_kr20_description/meshes/Link4.stl"
               meshscale="0.001 0.001 0.001" />
@@ -120,8 +120,8 @@
   <xacro:m_link_mesh name="${link_05_name}" color="LightGreen"
               origin_rpy="0 0 0" origin_xyz="0 0 0"
-              mass="157.633"
-              ixx="13.235" ixy="0" ixz="0"
-              iyy="13.235" iyz="0"
-              izz="9.655"
+              mass="2.38"
+              ixx="5.613" ixy="-0.8" ixz="0"
+              iyy="6.205" iyz="0"
+              izz="8.616"
               meshfile="package://kuka_kr20_description/meshes/Link5.stl"
               meshscale="0.001 0.001 0.001" />
@@ -133,8 +133,8 @@
   <xacro:m_link_mesh name="${link_06_name}" color="LightGreen"
               origin_rpy="0 0 0" origin_xyz="0 0 0"
-              mass="157.633"
-              ixx="13.235" ixy="0" ixz="0"
-              iyy="13.235" iyz="0"
-              izz="9.655"
+              mass="1.75"
+              ixx="2.865" ixy="0.01" ixz="0"
+              iyy="2.792" iyz="0"
+              izz="3.318"
               meshfile="package://kuka_kr20_description/meshes/Link6.stl"
               meshscale="0.001 0.001 0.001" />
@@ -146,21 +146,21 @@
   <xacro:m_link_mesh name="${link_07_name}" color="Grey"
               origin_rpy="0 0 0" origin_xyz="0 0 0"
-              mass="157.633"
-              ixx="13.235" ixy="0" ixz="0"
-              iyy="13.235" iyz="0"
-              izz="9.655"
+              mass="0.37"
+              ixx="0.2773" ixy="0" ixz="0"
+              iyy="0.493" iyz="0"
+              izz="0.2773"
               meshfile="package://kuka_kr20_description/meshes/Link7.stl"
               meshscale="0.001 0.001 0.001" />
    <xacro:m_joint name="q8" type="prismatic"
            axis_xyz="0 1 0"
-           origin_rpy="0 0 0" origin_xyz="0 -0.092 0"
+           origin_rpy="0 0 0" origin_xyz="0 -0.09 0"
            parent="${link_07_name}" child="${link_08_name}"
            limit_e="1000" limit_l="0" limit_u="0.1" limit_v="0.5" />
   <xacro:m_link_mesh name="${link_08_name}" color="Grey"
               origin_rpy="0 0 0" origin_xyz="0 0 0"
-              mass="157.633"
-              ixx="13.235" ixy="0" ixz="0"
-              iyy="13.235" iyz="0"
-              izz="9.655"
+              mass="1.69"
+              ixx="16.89" ixy="0" ixz="0"
+              iyy="0.5042" iyz="-0.28"
+              izz="16.89"
               meshfile="package://kuka_kr20_description/meshes/Link_EF.stl"
               meshscale="0.001 0.001 0.001" />
